File: echo.kicad_pcb (KiCad board)
At the start: 4 copper layers, 99 x 64 mm, 175 parts, among them J1 USB4215-03-A, J10 SS-52100-004, J2 D-SUB 9 Male, J3 MDC-036, J4 DC3RX19JA2, J5 0475710001, J6 104031-0811, J7 PJ-320D, J8 PJ-320D, J9 MDC-036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

Commit message: HW Rev 1.00
Parts:
- U8: value ~ -> MS9288A
- X1: value 24.576M -> 24.576 MHz
Routing:
- net /ESP_IO4: track 22.1 -> 20.9 mm
Other:
- outline, holes or cut-outs redrawn
- board text added: "${NAME}"
- board text added: "HDMI / REV ${VERSION}"
- board text added: "rh1.tech"
