File: usb_multiplexer.kicad_sch (KiCad schematic)
At the start: 3 parts, among them U11 TS3USB221RSER

Commit message: HW Rev 1.00
Connections:
- no-connect marks 1 -> 0
Changed lines of the file:
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@@
 	(title_block
 		(title "${NAME} ${MODEL}")
-		(date "2025-07-03")
+		(date "2025-07-04")
 		(rev "${VERSION}")
 		(company "Mikhail Matveev")
@@
 		(color 0 0 0 0)
 	)
-	(no_connect
-		(at 69.85 109.22)
-	)
 	(wire
