File: vga.kicad_sch (KiCad schematic)
At the start: 56 parts, among them J4 DC3RX19JA2, U6 AMS1117-3.3, U7 AMS1117-1.8, X1 24.576M

Commit message: HW Rev 1.00
Parts:
- U8: value ~ -> MS9288A
- X1: value 24.576M -> 24.576 MHz; symbol FRANK:Crystal,_25.576MHz -> FRANK:Crystal_25.576MHz; LCSC C9002 -> (none)
Changed lines of the file:
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@@
 	(title_block
 		(title "${NAME} ${MODEL}")
-		(date "2025-07-03")
+		(date "2025-07-04")
 		(rev "${VERSION}")
 		(company "Mikhail Matveev")
@@
 	)
 	(symbol
-		(lib_id "FRANK:Crystal,_25.576MHz")
+		(lib_id "FRANK:Crystal_25.576MHz")
 		(at 87.63 129.54 180)
 		(unit 1)
@@
 			)
 		)
-		(property "Value" "24.576M"
+		(property "Value" "24.576 MHz"
 			(at 87.63 127 0)
 			(effects
@@
 			)
 		)
-		(property "LCSC" "C9002"
+		(property "LCSC" ""
 			(at 87.63 129.54 0)
 			(effects
@@
 			)
 		)
-		(property "Value" "~"
+		(property "Value" "MS9288A"
 			(at 149.4633 130.81 0)
 			(effects
